Commit message: Repositioned camera.  Added some setup docs

File: henry_turret_description/urdf/henry_turret_description.urdf.xacro (robot description, xacro)
@@ -3,5 +3,5 @@
   <xacro:include filename="$(find zed_interfaces)/urdf/zed_descr.urdf.xacro"/>
   <joint name="zed_bracket_joint" type="fixed">
-    <origin xyz="0.089 0.089 0" rpy="0 0 0" />
+    <origin xyz="0.089 -0.089 0" rpy="0 0 0" />
     <parent link="world"/>
     <child link="zed_bracket_link" />

Commit message: Should be mostly written.  I'm sure there are lots of bugs.  Updated URDF and control script

File: henry_turret_description/urdf/henry_turret_description.urdf.xacro (robot description, xacro)
@@ -19,3 +19,9 @@
     <child link="zed_link" />
   </joint>
+  <link name="laser_link" />
+  <joint name="laser_joint" type="fixed">
+    <origin xyz="0 0 0.025" rpy="-1.57070 -1.5707 0" />
+    <parent link="hand_link"/>
+    <child link="laser_link" />
+  </joint>
 </robot>

Commit message: Added laser pointer and offline viewer to verify model

File: henry_turret_description/urdf/henry_turret_description.urdf.xacro (robot description, xacro)
@@ -19,5 +19,11 @@
     <child link="zed_link" />
   </joint>
-  <link name="laser_link" />
+  <link name="laser_link">
+    <visual>
+      <geometry>
+        <mesh filename="package://henry_turret_description/meshes/lp.dae"/>
+      </geometry>
+    </visual>
+  </link>
   <joint name="laser_joint" type="fixed">
     <origin xyz="0 0 0.025" rpy="-1.57070 -1.5707 0" />
